File: hardware/ecp5_soc_hat.sch (KiCad schematic (older format))
At the start: 31 parts, among them J1 DB15_Female_HighDensity_Mount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, J2 USB_A, U1 AS4C32M16SB, U2 74HC240, U3 LM2731XMF, X1 XO32, X3 HDR40, X4 HDR40

Commit message: Initial PCB placement
Signed-off-by: David Shah <davey1576@gmail.com>
Parts:
- C1, C11, C12, C13, C9: footprint Capacitor_SMD:C_0805_2012Metric_Pad1.33x1.40mm_HandSolder -> Capacitor_SMD:C_0805_2012Metric_Pad1.15x1.40mm_HandSolder
Changed lines of the file:
@@
 F 0 "C1" H 1142 3896 50  0000 L CNN
 F 1 "4.7µ" H 1142 3805 50  0000 L CNN
-F 2 "Capacitor_SMD:C_0805_2012Metric_Pad1.33x1.40mm_HandSolder" H 1050 3850 50  0001 C CNN
+F 2 "Capacitor_SMD:C_0805_2012Metric_Pad1.15x1.40mm_HandSolder" H 1050 3850 50  0001 C CNN
 F 3 "~" H 1050 3850 50  0001 C CNN
 	1    1050 3850
@@
 F 0 "C9" H 8242 1396 50  0000 L CNN
 F 1 "4.7µ" H 8242 1305 50  0000 L CNN
-F 2 "Capacitor_SMD:C_0805_2012Metric_Pad1.33x1.40mm_HandSolder" H 8150 1350 50  0001 C CNN
+F 2 "Capacitor_SMD:C_0805_2012Metric_Pad1.15x1.40mm_HandSolder" H 8150 1350 50  0001 C CNN
 F 3 "~" H 8150 1350 50  0001 C CNN
 	1    8150 1350
@@
 F 0 "C11" H 10342 1396 50  0000 L CNN
 F 1 "4.7µ" H 10342 1305 50  0000 L CNN
-F 2 "Capacitor_SMD:C_0805_2012Metric_Pad1.33x1.40mm_HandSolder" H 10250 1350 50  0001 C CNN
+F 2 "Capacitor_SMD:C_0805_2012Metric_Pad1.15x1.40mm_HandSolder" H 10250 1350 50  0001 C CNN
 F 3 "~" H 10250 1350 50  0001 C CNN
 	1    10250 1350
@@
 F 0 "C12" H 10642 1396 50  0000 L CNN
 F 1 "4.7µ" H 10642 1305 50  0000 L CNN
-F 2 "Capacitor_SMD:C_0805_2012Metric_Pad1.33x1.40mm_HandSolder" H 10550 1350 50  0001 C CNN
+F 2 "Capacitor_SMD:C_0805_2012Metric_Pad1.15x1.40mm_HandSolder" H 10550 1350 50  0001 C CNN
 F 3 "~" H 10550 1350 50  0001 C CNN
 	1    10550 1350
@@
 F 0 "C13" H 10942 1396 50  0000 L CNN
 F 1 "4.7µ" H 10942 1305 50  0000 L CNN
-F 2 "Capacitor_SMD:C_0805_2012Metric_Pad1.33x1.40mm_HandSolder" H 10850 1350 50  0001 C CNN
+F 2 "Capacitor_SMD:C_0805_2012Metric_Pad1.15x1.40mm_HandSolder" H 10850 1350 50  0001 C CNN
 F 3 "~" H 10850 1350 50  0001 C CNN
 	1    10850 1350

Commit message: PCB fully routed
Signed-off-by: David Shah <davey1576@gmail.com>
Parts:
- removed U2: 74HC240, Package_SO:SO-20_12.8x7.5mm_P1.27mm, symbol 74xx:74HC240
- added RN1, RN2: R_Pack04, Resistor_SMD:R_Array_Convex_4x0402, symbol Device:R_Pack04
- added U2: 74HC244, Package_SO:SO-20_12.8x7.5mm_P1.27mm, symbol 74xx:74HC244
- R2, R3, R4: value 270 -> DNP
Connections:
- net labels added: HS_BUF, VGA_BRIGHT, VGA_VB, VGA_VG, VGA_VR, VS_BUF
- net labels removed: EXPCON_CLKOUT
- wire segments 297 -> 313
Other:
- moved on the sheet: C8, J1

Commit message: Production PCBs rev1.0
Signed-off-by: David Shah <davey1576@gmail.com>
Parts:
- added J3: Conn_02x04_Odd_Even, Connector_PinHeader_2.54mm:PinHeader_2x04_P2.54mm_Vertical, symbol Connector_Generic:Conn_02x04_Odd_Even
Connections:
- net +3V3: now also J3.1 (Pin_1)
- net GND: now also J3.8 (Pin_8)
- net VGA_B: now also J3.4 (Pin_4)
- net VGA_BRIGHT: now also J3.3 (Pin_3)
- net VGA_G: now also J3.7 (Pin_7)
- net VGA_HS: now also J3.2 (Pin_2)
- net VGA_R: now also J3.5 (Pin_5)
- net VGA_VS: now also J3.6 (Pin_6)
- net EXPCON_OSC: no longer names the net of X3.29 (Pin_29)
- no-connect marks 20 -> 21
Changed lines of the file:
@@
 	1650 2100 1600 2100
-Wire Wire Line
-	1650 2300 1050 2300
 Wire Wire Line
 	1650 2400 1050 2400
@@
 Connection ~ 1600 2100
 Wire Wire Line
-	1600 2100 1050 2100
+	1600 2100 1100 2100
 NoConn ~ 1650 2000
 $Comp
@@
 	0    -1   -1   0
 $EndComp
-Text Label 1050 2300 0    50   ~ 0
-EXPCON_OSC
 Text Label 1050 2400 0    50   ~ 0
 EXPCON_CLKIN
@@
 Text Label 1050 2500 0    50   ~ 0
 VGA_BRIGHT
+Text Label 5550 6300 0    50   ~ 0
+VGA_R
+Wire Wire Line
+	5550 6300 6100 6300
+Text Label 5550 6400 0    50   ~ 0
+VGA_G
+Wire Wire Line
+	5550 6400 6100 6400
+Text Label 7150 6200 2    50   ~ 0
+VGA_B
+Text Label 7150 6100 2    50   ~ 0
+VGA_HS
+Text Label 7150 6300 2    50   ~ 0
+VGA_VS
+Wire Wire Line
+	7150 6300 6600 6300
+Wire Wire Line
+	6600 6100 7150 6100
+Wire Wire Line
+	7150 6200 6600 6200
+Text Label 5550 6200 0    50   ~ 0
+VGA_BRIGHT
+Wire Wire Line
+	5550 6200 6100 6200
+$Comp
+L power:GND #PWR01
+U 1 1 5BD62BD3
+P 6800 6550
+F 0 "#PWR01" H 6800 6300 50  0001 C CNN
+F 1 "GND" H 6805 6377 50  0000 C CNN
+F 2 "" H 6800 6550 50  0001 C CNN
+F 3 "" H 6800 6550 50  0001 C CNN
+	1    6800 6550
+	-1   0    0    -1
+$EndComp
+Wire Wire Line
+	6800 6550 6800 6400
+Wire Wire Line
+	6800 6400 6600 6400
+$Comp
+L power:+3V3 #PWR02
+U 1 1 5BD7CFB9
+P 5950 5900
+F 0 "#PWR02" H 5950 5750 50  0001 C CNN
+F 1 "+3V3" H 5965 6073 50  0000 C CNN
+F 2 "" H 5950 5900 50  0001 C CNN
+F 3 "" H 5950 5900 50  0001 C CNN
+	1    5950 5900
+	1    0    0    -1
+$EndComp
+Wire Wire Line
+	6100 6100 5950 6100
+Wire Wire Line
+	5950 6100 5950 5900
+$Comp
+L Connector_Generic:Conn_02x04_Odd_Even J3
+U 1 1 5BD98330
+P 6300 6200
+F 0 "J3" H 6350 6517 50  0000 C CNN
+F 1 "Conn_02x04_Odd_Even" H 6350 6426 50  0000 C CNN
+F 2 "Connector_PinHeader_2.54mm:PinHeader_2x04_P2.54mm_Vertical" H 6300 6200 50  0001 C CNN
+F 3 "~" H 6300 6200 50  0001 C CNN
+	1    6300 6200
+	1    0    0    -1
+$EndComp
+NoConn ~ 1650 2300
+$Comp
+L power:PWR_FLAG #FLG0101
+U 1 1 5BF5C8F4
+P 1000 1950
+F 0 "#FLG0101" H 1000 2025 50  0001 C CNN
+F 1 "PWR_FLAG" V 1000 2078 50  0000 L CNN
+F 2 "" H 1000 1950 50  0001 C CNN
+F 3 "~" H 1000 1950 50  0001 C CNN
+	1    1000 1950
+	0    -1   -1   0
+$EndComp
+Wire Wire Line
+	1000 1950 1100 1950
+Wire Wire Line
+	1100 1950 1100 2100
+Connection ~ 1100 2100
+Wire Wire Line
+	1100 2100 1050 2100
+$Comp
+L power:PWR_FLAG #FLG0102
+U 1 1 5BF77683
+P 2450 1900
+F 0 "#FLG0102" H 2450 1975 50  0001 C CNN
+F 1 "PWR_FLAG" V 2450 2028 50  0000 L CNN
+F 2 "" H 2450 1900 50  0001 C CNN
+F 3 "~" H 2450 1900 50  0001 C CNN
+	1    2450 1900
+	0    1    1    0
+$EndComp
+Wire Wire Line
+	2450 1900 2300 1900
+Connection ~ 2300 1900
+$Comp
+L power:PWR_FLAG #FLG0103
+U 1 1 5BF92F10
+P 9850 700
+F 0 "#FLG0103" H 9850 775 50  0001 C CNN
+F 1 "PWR_FLAG" H 9850 874 50  0000 C CNN
+F 2 "" H 9850 700 50  0001 C CNN
+F 3 "~" H 9850 700 50  0001 C CNN
+	1    9850 700
+	1    0    0    -1
+$EndComp
+Wire Wire Line
+	9850 700  9850 750
 $EndSCHEMATC
